File: rail_splitter.kicad_pcb (KiCad board)
At the start: 2 copper layers, 100 x 100 mm, 12 parts, among them J1 Screw_Terminal_01x02, U1 STM32F401RCTx

Commit message: v1 pcb
Parts:
- removed DS1: WC1602A - below, rail_lib:WC1602A - below
- added C1: 10n, Capacitor_SMD:C_1206_3216Metric, F.Cu at (90.0, 61.0)
- added C2: 0.22u, Capacitor_SMD:C_1206_3216Metric, F.Cu at (128.5, 78.0)
- added C3: 0.22u, Capacitor_SMD:C_1206_3216Metric, B.Cu at (110.5, 81.0)
- added C4: 100n, Capacitor_SMD:C_1206_3216Metric, F.Cu at (99.5, 130.0)
- added C5: 10u, Capacitor_SMD:C_1206_3216Metric, F.Cu at (99.2, 124.2)
- added D3: LED, LED_SMD:LED_1206_3216Metric, F.Cu at (102.4, 75.5)
- added D4: LED, LED_SMD:LED_1206_3216Metric, F.Cu at (93.4, 84.0)
- added J2: input -, Connector:Banana_Jack_1Pin, F.Cu at (61.5, 106.5)
- added J3: +load, Connector:Banana_Jack_1Pin, F.Cu at (139.0, 81.5)
- added J4: gnd load, Connector:Banana_Jack_1Pin, F.Cu at (139.5, 97.0)
- added J5: -load, Connector:Banana_Jack_1Pin, F.Cu at (139.5, 113.0)
- added J6: shunt+ display pos, Connector_PinHeader_1.00mm:PinHeader_1x02_P1.00mm_Vertical, F.Cu at (111.9, 68.0)
- added J7: shunt- display pos, Connector_PinHeader_1.00mm:PinHeader_1x01_P1.00mm_Vertical, F.Cu at (123.0, 68.5)
- added J8: shunt+ display neg, Connector_PinHeader_1.00mm:PinHeader_1x02_P1.00mm_Vertical, F.Cu at (125.5, 72.0)
- added J9: shunt- display neg, Connector_PinHeader_1.00mm:PinHeader_1x01_P1.00mm_Vertical, F.Cu at (139.0, 72.0)
- added Q1: PNP, Package_TO_SOT_SMD:SOT-23, F.Cu at (70.6, 73.0)
- added Q10: NPN, Package_TO_SOT_SMD:SOT-23, B.Cu at (118.0, 80.9)
- added Q11: NMOS, Package_TO_SOT_THT:TO-220-3_Vertical, F.Cu at (128.5, 61.0)
- added Q2: NPN, Package_TO_SOT_SMD:SOT-23, F.Cu at (88.5, 71.4)
- added Q3: NPN, Package_TO_SOT_SMD:SOT-23, F.Cu at (120.4, 88.0)
- added Q4: dar, Package_TO_SOT_THT:TO-220-3_Vertical, F.Cu at (78.4, 61.5)
- added Q5: NPN, Package_TO_SOT_SMD:SOT-23, F.Cu at (124.9, 88.0)
- added Q6: PNP, Package_TO_SOT_SMD:SOT-23, F.Cu at (126.1, 83.0)
- added Q7: PMOS, Package_TO_SOT_THT:TO-220-3_Vertical, F.Cu at (114.4, 61.0)
- added Q8: PNP, Package_TO_SOT_SMD:SOT-23, B.Cu at (126.8, 102.6)
- added Q9: PNP, Package_TO_SOT_SMD:SOT-23, B.Cu at (131.4, 102.5)
- added Qdar1: PNP, Package_TO_SOT_THT:TO-220-3_Vertical, F.Cu at (97.5, 61.0)
- added R1: 0.33, Resistor_SMD:R_2512_6332Metric, F.Cu at (94.0, 67.5)
- added R10: R, Resistor_SMD:R_1206_3216Metric, F.Cu at (123.0, 74.5)
- added R11: R, Resistor_SMD:R_1206_3216Metric, F.Cu at (105.5, 78.5)
- added R12: R, Resistor_SMD:R_1206_3216Metric, F.Cu at (114.0, 84.0)
- added R13: R, Resistor_SMD:R_1206_3216Metric, F.Cu at (120.0, 84.0)
- added R14: R, Resistor_SMD:R_1206_3216Metric, F.Cu at (122.5, 92.5)
- added R15: R, Resistor_SMD:R_1206_3216Metric, F.Cu at (130.5, 83.5)
- added R16: R, Resistor_SMD:R_1206_3216Metric, F.Cu at (115.5, 90.5)
- added R17: R, Resistor_SMD:R_1206_3216Metric, F.Cu at (106.0, 89.0)
- added R18: R, Resistor_SMD:R_1206_3216Metric, F.Cu at (111.5, 89.0)
- added R19: R, Resistor_SMD:R_1206_3216Metric, F.Cu at (111.5, 95.0)
- added R2: 0.33, Resistor_SMD:R_2512_6332Metric, F.Cu at (102.5, 67.5)
- added R20: R, Resistor_SMD:R_2512_6332Metric, B.Cu at (131.0, 72.0)
- added R21: R, Resistor_SMD:R_1206_3216Metric, B.Cu at (123.5, 76.5)
- added R22: R, Resistor_SMD:R_1206_3216Metric, B.Cu at (131.0, 78.0)
- added R23: R, Resistor_SMD:R_1206_3216Metric, B.Cu at (133.0, 88.5)
- added R24: R, Resistor_SMD:R_1206_3216Metric, B.Cu at (126.5, 84.5)
- added R25: R, Resistor_SMD:R_1206_3216Metric, B.Cu at (132.5, 93.0)
- added R26: R, Resistor_SMD:R_1206_3216Metric, B.Cu at (131.0, 83.0)
- added R27: R, Resistor_SMD:R_1206_3216Metric, B.Cu at (122.0, 101.5)
- added R28: R, Resistor_SMD:R_1206_3216Metric, B.Cu at (110.5, 86.5)
- added R29: R, Resistor_SMD:R_1206_3216Metric, B.Cu at (106.0, 81.0)
- added R3: 67, Resistor_SMD:R_1206_3216Metric, F.Cu at (63.5, 73.0)
- added R30: R, Resistor_SMD:R_1206_3216Metric, B.Cu at (117.0, 88.5)
- added R31: R, Resistor_SMD:R_1206_3216Metric, B.Cu at (120.5, 70.5)
- added R32: R, Resistor_SMD:R_1206_3216Metric, B.Cu at (138.0, 62.0)
- added R33: R, Resistor_SMD:R_1206_3216Metric, B.Cu at (130.0, 56.0)
- added R34: 1k, Resistor_SMD:R_1206_3216Metric, F.Cu at (90.0, 99.0)
- added R35: 1k, Resistor_SMD:R_1206_3216Metric, F.Cu at (97.5, 80.0)
- added R36: 1k, Resistor_SMD:R_1206_3216Metric, F.Cu at (101.0, 88.5)
- added R37: 1k, Resistor_SMD:R_1206_3216Metric, F.Cu at (102.0, 92.5)
- added R38: 1k, Resistor_SMD:R_1206_3216Metric, F.Cu at (99.0, 84.0)
- added R4: 5.6k, Resistor_SMD:R_1206_3216Metric, F.Cu at (69.5, 78.0)
- added R5: 3.3k, Resistor_SMD:R_1206_3216Metric, F.Cu at (75.5, 73.0)
- added R6: 1k, Resistor_SMD:R_1206_3216Metric, F.Cu at (82.0, 86.5)
- added R7: 470, Resistor_SMD:R_1206_3216Metric, F.Cu at (79.0, 86.5)
- added R8: R, Resistor_SMD:R_2512_6332Metric, F.Cu at (117.5, 68.5)
- added R9: R, Resistor_SMD:R_1206_3216Metric, F.Cu at (110.0, 75.5)
- added RV4: R_Potentiometer, Potentiometer_SMD:Potentiometer_ACP_CA6-VSMD_Vertical, F.Cu at (99.0, 105.3)
- added SW1: SW_Push, Button_Switch_THT:SW_PUSH_6mm_H4.3mm, F.Cu at (137.0, 127.5)
- added SW2: SW_Push, Button_Switch_THT:SW_PUSH_6mm_H4.3mm, F.Cu at (130.2, 132.5)
- added U2: NE5532, Package_SO:SOIC-8_3.9x4.9mm_P1.27mm, F.Cu at (115.5, 77.1)
- added U3: NE5532, Package_SO:SOIC-8_3.9x4.9mm_P1.27mm, B.Cu at (126.5, 92.4)
- added U4: NE5532, Package_SO:SOIC-8_3.9x4.9mm_P1.27mm, B.Cu at (116.1, 100.5)
- added U5: LM2936-3.3, Package_TO_SOT_SMD:SOT-223-3_TabPin2, F.Cu at (99.1, 116.7)
- added U6: NE5532, Package_SO:SOIC-8_3.9x4.9mm_P1.27mm, F.Cu at (95.0, 90.1)
- D1, D2: value 1N4148W -> 1N4148WT; footprint Diode_SMD:D_SOD-123 -> Diode_SMD:D_SOD-523; moved to F.Cu
- J1: value Screw_Terminal_01x02 -> input +; footprint TerminalBlock_Phoenix:TerminalBlock_Phoenix_MKDS-3-2-5.08_1x02_P5.08mm_Horizontal -> Connector:Banana_Jack_1Pin; moved to F.Cu
- RV1: value R_Potentiometer -> 1k; footprint PID_lib:front_plate_pot -> Potentiometer_SMD:Potentiometer_ACP_CA6-VSMD_Vertical
- U1: value STM32F401RCTx -> OP07; footprint Package_QFP:LQFP-64_10x10mm_P0.5mm -> Package_SO:SOIC-8_3.9x4.9mm_P1.27mm; moved to F.Cu
- moved D2 54.0 mm to (61.8, 78.0), turned to 180 degrees
- moved U1 53.9 mm to (80.9, 95.0), turned to -90 degrees
- moved D1 49.6 mm to (65.2, 78.0), turned to 180 degrees
- moved RV1 47.8 mm to (82.0, 77.7), turned to -90 degrees
- moved J1 45.0 mm to (61.0, 87.5)
- moved RV2 17.5 mm to (82.5, 124.5)
- moved RV3 9.53 mm to (115.5, 124.2)
Connections:
- D2 pad 1: Net-(D2-K) -> Net-(D1-A)
- D2 pad 2: Net-(D1-K) -> VCC
- J1 pad 1: Net-(J1-Pin_1) -> VCC
- RV1 pad 1: unconnected-(RV1-Pad1) -> Net-(Q2-B)
- RV1 pad 2: unconnected-(RV1-Pad2) -> Net-(R6-Pad1)
- RV2 pad 1: unconnected-(RV2-Pad1) -> +VCC OUTPUT
- RV2 pad 2: unconnected-(RV2-Pad2) -> Net-(U1-+)
- RV2 pad 3: unconnected-(RV2-Pad3) -> Net-(J1-Pin_1)
- RV3 pad 1: unconnected-(RV3-Pad1) -> GNDD
- RV3 pad 2: unconnected-(RV3-Pad2) -> Limit
- RV3 pad 3: unconnected-(RV3-Pad3) -> +3.3V
- U1 pad 2: unconnected-(U1-PC13-Pad2) -> GND
- U1 pad 3: unconnected-(U1-PC14-Pad3) -> Net-(U1-+)
- U1 pad 4: unconnected-(U1-PC15-Pad4) -> VEE
- U1 pad 6: unconnected-(U1-PH1-Pad6) -> Net-(Q1-C)
- U1 pad 7: unconnected-(U1-NRST-Pad7) -> VCC
Routing:
- net GND: track 0.00 -> 298.7 mm, vias 0 -> 2
- net VEE: track 0.00 -> 97.7 mm, vias 0 -> 3
- net Net-(Q1-C): track 0.00 -> 83.0 mm
- net Net-(U2B-+): track 0.00 -> 79.6 mm, vias 0 -> 4
- net Net-(Q9-B): track 0.00 -> 72.9 mm
- net Limit: track 0.00 -> 70.7 mm, vias 0 -> 1
- net Net-(J5-Pin_1): track 0.00 -> 62.3 mm
- net Net-(Q5-B): track 0.00 -> 61.5 mm, vias 0 -> 1
- net Net-(Q2-E): track 0.00 -> 56.2 mm
- net GNDD: track 0.00 -> 54.3 mm, vias 0 -> 1
- net Net-(Q7-G): track 0.00 -> 42.9 mm
- net +3.3V: track 0.00 -> 41.5 mm, vias 0 -> 1
- net Net-(U3A-+): track 0.00 -> 36.6 mm
- net Net-(U1-+): track 0.00 -> 36.3 mm, vias 0 -> 2
- net Net-(R31-Pad1): track 0.00 -> 33.9 mm
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- added copper zone on F.Cu, net VCC
- added copper zone on B.Cu, net VEE
Other:
- board text added: "Current limit"
- board text removed: "Negative current limit"
- board text removed: "Positive current limit"
