File: rail_splitter.kicad_sch (KiCad schematic)
At the start: 13 parts, among them J1 Screw_Terminal_01x02, Q1 NPN, Q2 PNP, U1 STM32F401RCTx

Commit message: v1 pcb
Parts:
- removed D1, D2: 1N4148W, Diode_SMD:D_SOD-123, symbol Diode:1N4148W
- removed H1, H2, H3, H4: MountingHole, PID_lib:M3_hole_with_spacer, symbol Mechanical:MountingHole
- removed J1: Screw_Terminal_01x02, TerminalBlock_Phoenix:TerminalBlock_Phoenix_MKDS-3-2-5.08_1x02_P5.08mm_Horizontal, symbol Connector:Screw_Terminal_01x02
- removed Q1: NPN, symbol Simulation_SPICE:NPN
- removed Q2: PNP, symbol Simulation_SPICE:PNP
- removed U1: STM32F401RCTx, Package_QFP:LQFP-64_10x10mm_P0.5mm, symbol MCU_ST_STM32F4:STM32F401RCTx
- added C1: 10n, Capacitor_SMD:C_1206_3216Metric, symbol Device:C
- added C2, C3: 0.22u, Capacitor_SMD:C_1206_3216Metric, symbol Device:C
- added C4: 100n, Capacitor_SMD:C_1206_3216Metric, symbol Device:C
- added C5: 10u, Capacitor_SMD:C_1206_3216Metric, symbol Device:C
- added D1, D2: 1N4148WT, Diode_SMD:D_SOD-523, symbol Diode:1N4148WT
- added D3, D4: LED, LED_SMD:LED_1206_3216Metric, symbol Device:LED
- added J1: input +, Connector:Banana_Jack_1Pin, symbol Connector:Conn_01x01_Socket
- added J2: input -, Connector:Banana_Jack_1Pin, symbol Connector:Conn_01x01_Socket
- added J3: +load, Connector:Banana_Jack_1Pin, symbol Connector:Conn_01x01_Socket
- added J4: gnd load, Connector:Banana_Jack_1Pin, symbol Connector:Conn_01x01_Socket
- added J5: -load, Connector:Banana_Jack_1Pin, symbol Connector:Conn_01x01_Socket
- added J6: shunt+ display pos, Connector_PinHeader_1.00mm:PinHeader_1x02_P1.00mm_Vertical, symbol Connector:Conn_01x01_Socket
- added J7: shunt- display pos, Connector_PinHeader_1.00mm:PinHeader_1x01_P1.00mm_Vertical, symbol Connector:Conn_01x01_Socket
- added J8: shunt+ display neg, Connector_PinHeader_1.00mm:PinHeader_1x02_P1.00mm_Vertical, symbol Connector:Conn_01x01_Socket
- added J9: shunt- display neg, Connector_PinHeader_1.00mm:PinHeader_1x01_P1.00mm_Vertical, symbol Connector:Conn_01x01_Socket
- added Q1, Q6, Q8, Q9: PNP, Package_TO_SOT_SMD:SOT-23, symbol Simulation_SPICE:PNP
- added Q10, Q2, Q3, Q5: NPN, Package_TO_SOT_SMD:SOT-23, symbol Simulation_SPICE:NPN
- added Q11: NMOS, Package_TO_SOT_THT:TO-220-3_Vertical, symbol Simulation_SPICE:NMOS
- added Q4: dar, Package_TO_SOT_THT:TO-220-3_Vertical, symbol Simulation_SPICE:NPN
- added Q7: PMOS, Package_TO_SOT_THT:TO-220-3_Vertical, symbol Simulation_SPICE:PMOS
- added Qdar1: PNP, Package_TO_SOT_THT:TO-220-3_Vertical, symbol Simulation_SPICE:PNP
- added R1, R2: 0.33, Resistor_SMD:R_2512_6332Metric, symbol Device:R
- added R10, R11, R12, R13, R14, R15, R16, R17, R18, R19, R21, R22, R23, R24, R25, R26, R27, R28, R29, R30, R31, R32, R33, R9: R, Resistor_SMD:R_1206_3216Metric, symbol Device:R
- added R20, R8: R, Resistor_SMD:R_2512_6332Metric, symbol Device:R
- added R3: 67, Resistor_SMD:R_1206_3216Metric, symbol Device:R
- added R34, R35, R36, R37, R38, R6: 1k, Resistor_SMD:R_1206_3216Metric, symbol Device:R
- added R4: 5.6k, Resistor_SMD:R_1206_3216Metric, symbol Device:R
- added R5: 3.3k, Resistor_SMD:R_1206_3216Metric, symbol Device:R
- added R7: 470, Resistor_SMD:R_1206_3216Metric, symbol Device:R
- added RV4: R_Potentiometer, Potentiometer_SMD:Potentiometer_ACP_CA6-VSMD_Vertical, symbol Device:R_Potentiometer
- added SW1, SW2: SW_Push, Button_Switch_THT:SW_PUSH_6mm_H4.3mm, symbol Switch:SW_Push
- added U1: OP07, Package_SO:SOIC-8_3.9x4.9mm_P1.27mm, symbol Amplifier_Operational:OP07
- added U2, U3, U4, U6: NE5532, Package_SO:SOIC-8_3.9x4.9mm_P1.27mm, symbol Amplifier_Operational:NE5532
- added U5: LM2936-3.3, Package_TO_SOT_SMD:SOT-223-3_TabPin2, symbol Regulator_Linear:LM2936-3.3
- RV1: value R_Potentiometer -> 1k; footprint PID_lib:front_plate_pot -> Potentiometer_SMD:Potentiometer_ACP_CA6-VSMD_Vertical
- RV2: value R_Potentiometer -> ~; footprint PID_lib:front_plate_pot -> Potentiometer_THT:Potentiometer_Alps_RK09Y11_Single_Horizontal
- RV3: footprint PID_lib:front_plate_pot -> Potentiometer_SMD:Potentiometer_ACP_CA6-VSMD_Vertical
Connections:
- net GND: now also D3.1 (K), J4.1 (Pin_1), Q3.3 (E), Q5.3 (E), Q8.1 (C), Q9.1 (C), R1.2, R19.2, R2.1, R23.2, R32.1, R35.2, R36.1, R38.2, SW1.1, SW2.1, U1.2 (-), U3.5 (+)
- net at RV1.1: now also Q2.2 (B), R5.2
- net at RV1.2: now also R6.1
- net VCC: now reaches RV2.1
- net VCC: now also C2.1, C4.1, D2.2 (A), J1.1 (Pin_1), Q4.1 (C), Q6.3 (E), Q7.3 (S), R15.1, R3.1, U1.7 (V+), U2.8 (V+), U3.8 (V+), U4.8 (V+), U5.1 (VI), U6.8 (V+)
- net at RV2.2: now also R34.1, U1.3 (+)
- net VEE: now reaches RV2.3
- net VEE: now also C3.1, J2.1 (Pin_1), Q10.3 (E), Q11.3 (S), Qdar1.1 (C), R29.2, R4.2, R7.2, U1.4 (V-), U2.4 (V-), U3.4 (V-), U4.4 (V-), U6.4 (V-)
- net +3.3V: now reaches RV3.1
- net +3.3V: now also C5.1, RV4.1, U5.3 (VO)
- net Limit: now reaches RV3.2
- net Limit: now also U2.6 (-), U4.3 (+)
- net GNDD: now reaches RV3.3
- net GNDD: now also C4.2, C5.2, RV4.3, U5.2 (GND)
- new net: R34.2, R35.1, U6.3 (+)
- new net: Qdar1.3 (E), R2.2
- new net: R37.2, U6.1, U6.5 (+)
- new net: RV4.2, U6.6 (-)
- new net: D4.2 (A), U6.7
- new net: J8.1 (Pin_1), Q11.1 (D), R20.2, R21.2
- new net: Q9.2 (B), R30.1, SW2.2
- new net: R22.2, R26.1, U3.2 (-)
- new net: R24.1, R26.2, U3.1
- new net: R31.1, R32.2, R33.1
- new net: Q11.2 (G), R33.2
- new net: C1.1, Q1.1 (C), Q2.1 (C), Q4.2 (B), R5.1, U1.6
- new net: Q4.3 (E), R1.1
- new net: Q3.1 (C), Q5.1 (C), R14.2
- new net: Q3.2 (B), R13.2
- new net: Q10.1 (C), R30.2, R31.2
- new net: C3.2, Q10.2 (B), R28.2, R29.1
- new net: J6.1 (Pin_1), Q7.1 (D), R8.1, R9.1
- new net: Q7.2 (G), R17.1
- new net: R24.2, R25.1, U3.6 (-)
- new net: C2.2, Q6.2 (B), R14.1, R15.2
- new net: R17.2, R18.2, R19.1
- new net: D3.2 (A), R11.2
- new net: Q8.2 (B), R27.1
- new net: Q8.3 (E), Q9.3 (E), R28.1
- new net: D4.1 (K), R38.1
- new net: Q6.1 (C), R16.1, R18.1
- new net: Q5.2 (B), R16.2, SW1.2
- new net: R12.2, R13.1, R25.2, U2.1, U2.5 (+), U2.7, U3.7, U4.2 (-)
- new net: D1.1 (K), Q1.2 (B), R4.1
- new net: J5.1 (Pin_1), J9.1 (Pin_1), R20.1, R22.1
- new net: R11.1, R9.2, U2.3 (+)
- new net: J3.1 (Pin_1), J7.1 (Pin_1), R10.1, R8.2
- new net: C1.2, Q2.3 (E), Qdar1.2 (B), R6.2, R7.1
- new net: R27.2, U4.1
- new net: R21.1, R23.1, U3.3 (+)
- new net: R10.2, R12.1, U2.2 (-)
- new net: D1.2 (A), D2.1 (K)
- new net: Q1.3 (E), R3.2
- new net: R36.2, R37.1, U6.2 (-)
